File: hardware/mcu.kicad_sch (KiCad schematic)
At the start: 1 part

Commit message: MCU module is completed
Parts:
- added C? (x6): 100nF, symbol Device:C_Small
- added C?: 1uF/10V, symbol Device:C_Polarized_Small
- added C? (x2): 1uF/6V, symbol Device:C_Polarized_Small
- added C? (x2): 20pF, symbol Device:C_Small
- added J?: BOOT, symbol Connector:Conn_01x02_Male
- added R? (x2): 100K, symbol Device:R_Small
- added R?: 100R, symbol Device:R_Small
- added Y?: 32KHz, symbol Device:Crystal_Small
- added Y?: 8MHz, symbol Device:Crystal_Small
Connections:
- net at U?.1 (VBAT): now also C?.1
- net DISP_A: now reaches U?.13 (PA3)
- net DISP_B: now reaches U?.14 (PA4)
- net DISP_C: now reaches U?.15 (PA5)
- net DISP_D: now reaches U?.16 (PA6)
- net DISP_E: now reaches U?.17 (PA7)
- net DISP_F: now reaches U?.18 (PB0)
- net DISP_G: now reaches U?.19 (PB1)
- net DISP_P: now reaches U?.20 (PB2)
- net GND: now reaches U?.23 (VSS)
- net GND: now also U?.35 (VSS), U?.47 (VSS), U?.8 (VSSA), C?.1, C?.1, C?.2, C?.2, C?.2, C?.2, C?.2, C?.2, C?.2, C?.2, C?.2, R?.2
- net +3V3: now reaches U?.24 (VDD)
- net +3V3: now also U?.36 (VDD), U?.48 (VDD), C?.1, C?.1, C?.1, C?.1, C?.1, J?.1 (Pin_1), R?.1, R?.2
- net RELAY: now reaches U?.28 (PB15)
- net FLOW: now reaches U?.29 (PA8)
- net RCC_OSC32_IN: now reaches U?.3 (PC14)
- net RCC_OSC32_IN: now also Y?.2
- net BUZZER: now reaches U?.30 (PA9)
- net RCC_OSC32_OUT: now reaches U?.4 (PC15)
- net RCC_OSC32_OUT: now also Y?.1
- net BTN_IO: now reaches U?.41 (PB5)
- net BTN_START: now reaches U?.42 (PB6)
- net BTN_MODE: now reaches U?.43 (PB7)
- net RCC_OSC_IN: now reaches U?.5 (PD0)
- net RCC_OSC_IN: now also C?.2, Y?.2
- net RCC_OSC_OUT: now reaches U?.6 (PD1)
- net RCC_OSC_OUT: now also C?.2, Y?.1
- net nRESET: now reaches U?.7 (NRST)
- net nRESET: now also C?.1, R?.1
- net at U?.9 (VDDA): now also C?.1, C?.1, R?.2
- new net BOOT0: J?.2 (Pin_2), R?.1
Other:
- note added: "Boot"
- note added: "Crystal Oscillators"
- note added: "Reset"
