File: hardware/power.kicad_sch (KiCad schematic)
At the start: 16 parts, among them U4 TPS7A4901DGNT, U5 LD1085D2M-R

Commit message: yeni seyler eklendi
Parts:
- removed C20: 100uF/35V, Capacitor_SMD:CP_Elec_10x10.5, symbol Device:CP
- removed R23: 1K, Resistor_SMD:R_0603_1608Metric, symbol Device:R
- removed R24: 33, Resistor_SMD:R_0603_1608Metric, symbol Device:R
- removed R25: 120, Resistor_SMD:R_0603_1608Metric, symbol Device:R
- removed U5: LD1085D2M-R, Power:LD1085D2M-R, symbol LD1085D2MR:LD1085D2M-R
Connections:
- net VCC is gone; now on net +12V: F1.2
- net +12V: no longer C19.1, U4.5 (EN), U4.8 (IN)
- net at C16.1, D4.1 (K): now also C19.1, U4.5 (EN), U4.8 (IN)
Other:
- company: AKIM Elektronik LTD. STI. -> (none)
- title: KAPAK/VANA KONTROL KARTI -> MilkPompPower
- moved on the sheet: C15, C16, C17, C18, C19, D4, F1, R20, R21, R22, U4
